File: PCB/Devboard.kicad_sch (KiCad schematic)
At the start: 21 parts, among them J1 USB_C_Receptacle_USB2.0_14P, U1 RP2040, U2 NCP1117-3.3_SOT223

Commit message: schematic done
Parts:
- removed U2: NCP1117-3.3_SOT223, Package_TO_SOT_SMD:SOT-223-3_TabPin2, symbol Regulator_Linear:NCP1117-3.3_SOT223
- added C15, C16: 33pF, Capacitor_SMD:C_0603_1608Metric, symbol Device:C
- added C17: 0.1uF, Capacitor_SMD:C_0402_1005Metric, symbol Device:C
- added J2, J3: Conn_01x20, Connector_PinHeader_2.54mm:PinHeader_1x20_P2.54mm_Vertical, symbol Connector_Generic:Conn_01x20
- added J4: Conn_01x03, Connector_PinHeader_2.54mm:PinHeader_1x03_P2.54mm_Vertical, symbol Connector_Generic:Conn_01x03
- added R5, R6: 1K, Resistor_SMD:R_0402_1005Metric, symbol Device:R
- added R7: 10K, Resistor_SMD:R_0402_1005Metric, symbol Device:R
- added SW1: SW_Push, Button_Switch_SMD:SW_Push_SPST_NO_Alps_SKRK, symbol Switch:SW_Push
- added U2: MCP1700x-330xxTT, Package_TO_SOT_SMD:SOT-23, symbol Regulator_Linear:MCP1700x-330xxTT
- added U3: W25Q128JVS, Package_SON:Winbond_USON-8-1EP_3x2mm_P0.5mm_EP0.2x1.6mm, symbol Memory_Flash:W25Q16JVSS
- added Y1: 12 MHz, Crystal:Crystal_SMD_3225-4Pin_3.2x2.5mm, symbol Device:Crystal_GND24
- C1, C10, C11, C12, C2, C3, C4, C5, C6, C7, C8, C9: footprint (none) -> Capacitor_SMD:C_0402_1005Metric
- C13, C14: footprint (none) -> Capacitor_SMD:C_0603_1608Metric
- J1: footprint (none) -> Connector_USB:USB_C_Receptacle_HRO_TYPE-C-31-M-12
- R1, R2, R3, R4: footprint (none) -> Resistor_SMD:R_0402_1005Metric
Connections:
- net +3V3: now also C17.1, J3.5 (Pin_5), R7.1, U2.2 (VO), U3.8 (VCC)
- net GND: now also U1.19 (TESTEN), C15.2, C16.1, C17.2, J2.13 (Pin_13), J2.18 (Pin_18), J2.3 (Pin_3), J2.8 (Pin_8), J3.13 (Pin_13), J3.18 (Pin_18), J3.3 (Pin_3), J3.8 (Pin_8), J4.2 (Pin_2), SW1.1, U2.1 (GND), U3.4 (GND), Y1.2, Y1.4
- net VBUS: now also J3.1 (Pin_1), U2.3 (VI)
- net XIN: now also C15.1, Y1.3
- net XOUT: now also R5.2
- net GPIO8: now reaches U1.11 (GPIO8)
- net GPIO8: now also J2.11 (Pin_11)
- net GPIO9: now reaches U1.12 (GPIO9)
- net GPIO9: now also J2.12 (Pin_12)
- net GPIO10: now reaches U1.13 (GPIO10)
- net GPIO10: now also J2.14 (Pin_14)
- net GPIO11: now reaches U1.14 (GPIO11)
- net GPIO11: now also J2.15 (Pin_15)
- net GPIO12: now reaches U1.15 (GPIO12)
- net GPIO12: now also J2.16 (Pin_16)
- net GPIO13: now reaches U1.16 (GPIO13)
- net GPIO13: now also J2.17 (Pin_17)
- net GPIO14: now reaches U1.17 (GPIO14)
- net GPIO14: now also J2.19 (Pin_19)
- net GPIO15: now reaches U1.18 (GPIO15)
- net GPIO15: now also J2.20 (Pin_20)
- net GPIO0: now reaches U1.2 (GPIO0)
- net GPIO0: now also J2.1 (Pin_1)
- net SWCLK: now reaches U1.24 (SWCLK)
- net SWCLK: now also J4.1 (Pin_1)
- net SWD: now reaches U1.25 (SWD)
- net SWD: now also J4.3 (Pin_3)
- net RUN: now reaches U1.26 (RUN)
- net RUN: now also J3.11 (Pin_11)
- net GPIO16: now reaches U1.27 (GPIO16)
- net GPIO16: now also J3.20 (Pin_20)
- net GPIO17: now reaches U1.28 (GPIO17)
- net GPIO17: now also J3.19 (Pin_19)
- net GPIO18: now reaches U1.29 (GPIO18)
- net GPIO18: now also J3.17 (Pin_17)
- net GPIO1: now reaches U1.3 (GPIO1)
- net GPIO1: now also J2.2 (Pin_2)
- net GPIO19: now reaches U1.30 (GPIO19)
- net GPIO19: now also J3.16 (Pin_16)
- net GPIO20: now reaches U1.31 (GPIO20)
- net GPIO20: now also J3.15 (Pin_15)
- net GPIO21: now reaches U1.32 (GPIO21)
- net GPIO21: now also J3.14 (Pin_14)
- net GPIO22: now reaches U1.34 (GPIO22)
- net GPIO22: now also J3.12 (Pin_12)
- net GPIO23: now reaches U1.35 (GPIO23)
- net GPIO23: now also J3.10 (Pin_10)
- net GPIO24: now reaches U1.36 (GPIO24)
- net GPIO24: now also J3.9 (Pin_9)
- net GPIO26_ADC0: now reaches U1.38 (GPIO26_ADC0)
- net GPIO26_ADC0: now also J3.7 (Pin_7)
- net GPIO27_ADC1: now reaches U1.39 (GPIO27_ADC1)
- net GPIO27_ADC1: now also J3.6 (Pin_6)
- net GPIO2: now reaches U1.4 (GPIO2)
- net GPIO2: now also J2.4 (Pin_4)
- net GPIO28_ADC2: now reaches U1.40 (GPIO28_ADC2)
- net GPIO28_ADC2: now also J3.4 (Pin_4)
- net GPIO29_ADC3: now reaches U1.41 (GPIO29_ADC3)
- net GPIO29_ADC3: now also J3.2 (Pin_2)
- net GPIO3: now reaches U1.5 (GPIO3)
- net GPIO3: now also J2.5 (Pin_5)
- net QSPI_SD3: now reaches U1.51 (QSPI_SD3)
- net QSPI_SD3: now also U3.7 (~{HOLD}/~{RESET}/IO_{3})
- net QSPI_SCLK: now reaches U1.52 (QSPI_SCLK)
- net QSPI_SCLK: now also U3.6 (CLK)
- net QSPI_SD0: now reaches U1.53 (QSPI_SD0)
- net QSPI_SD0: now also U3.5 (DI/IO_{0})
- net QSPI_SD2: now reaches U1.54 (QSPI_SD2)
- net QSPI_SD2: now also U3.3 (~{WP}/IO_{2})
- net QSPI_SD1: now reaches U1.55 (QSPI_SD1)
- net QSPI_SD1: now also U3.2 (DO/IO_{1})
- net QSPI_SS: now reaches U1.56 (QSPI_SS)
- net QSPI_SS: now also R6.2, R7.2, U3.1 (~{CS})
- net GPIO4: now reaches U1.6 (GPIO4)
- net GPIO4: now also J2.6 (Pin_6)
- net GPIO5: now reaches U1.7 (GPIO5)
- net GPIO5: now also J2.7 (Pin_7)
- net GPIO6: now reaches U1.8 (GPIO6)
- net GPIO6: now also J2.9 (Pin_9)
- net GPIO7: now reaches U1.9 (GPIO7)
- net GPIO7: now also J2.10 (Pin_10)
- new net: C16.2, R5.1, Y1.1
- new net: R6.1, SW1.2
- no-connect marks 0 -> 1

Commit message: pcb image fix
Changed lines of the file:
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@@
 	)
 	(junction
+		(at 66.04 57.15)
+		(diameter 0)
+		(color 0 0 0 0)
+	)
+	(junction
 		(at 77.47 58.42)
 		(diameter 0)
@@
 	)
 	(junction
-		(at 64.77 57.15)
-		(diameter 0)
-		(color 0 0 0 0)
-	)
-	(junction
 		(at 55.88 69.85)
 		(diameter 0)
@@
 	(wire
 		(pts
+			(xy 66.04 54.61) (xy 64.77 54.61)
+		)
+		(stroke
+			(width 0)
+			(type default)
+		)
+	)
+	(wire
+		(pts
 			(xy 251.46 106.68) (xy 256.54 106.68)
 		)
@@
 	(wire
 		(pts
-			(xy 64.77 54.61) (xy 64.77 57.15)
+			(xy 66.04 54.61) (xy 66.04 57.15)
 		)
 		(stroke
@@
 	(wire
 		(pts
-			(xy 64.77 57.15) (xy 64.77 58.42)
+			(xy 69.85 58.42) (xy 77.47 58.42)
 		)
 		(stroke
@@
 	(wire
 		(pts
-			(xy 69.85 58.42) (xy 77.47 58.42)
+			(xy 104.14 50.8) (xy 115.57 50.8)
 		)
 		(stroke
@@
 	(wire
 		(pts
-			(xy 104.14 50.8) (xy 115.57 50.8)
+			(xy 208.28 129.54) (xy 208.28 116.84)
 		)
 		(stroke
@@
 	(wire
 		(pts
-			(xy 208.28 129.54) (xy 208.28 116.84)
+			(xy 15.24 124.46) (xy 15.24 125.73)
 		)
 		(stroke
@@
 	(wire
 		(pts
-			(xy 15.24 124.46) (xy 15.24 125.73)
+			(xy 102.87 68.58) (xy 104.14 68.58)
 		)
 		(stroke
@@
 	(wire
 		(pts
-			(xy 102.87 68.58) (xy 104.14 68.58)
+			(xy 66.04 57.15) (xy 64.77 57.15)
 		)
 		(stroke
@@
 	(wire
 		(pts
+			(xy 66.04 57.15) (xy 66.04 58.42)
+		)
+		(stroke
+			(width 0)
+			(type default)
+		)
+	)
+	(wire
+		(pts
 			(xy 102.87 99.06) (xy 104.14 99.06)
 		)
@@
 	(symbol
 		(lib_id "power:GND")
-		(at 64.77 58.42 0)
+		(at 66.04 58.42 0)
 		(unit 1)
 		(exclude_from_sim no)
@@
 		(dnp no)
 		(property "Reference" "#PWR09"
-			(at 64.77 64.77 0)
+			(at 66.04 64.77 0)
 			(effects
 				(font
@@
 		)
 		(property "Value" "GND"
-			(at 68.326 60.452 0)
+			(at 69.596 60.452 0)
 			(effects
 				(font
@@
 		)
 		(property "Footprint" ""
-			(at 64.77 58.42 0)
+			(at 66.04 58.42 0)
 			(effects
 				(font
@@
 		)
 		(property "Datasheet" ""
-			(at 64.77 58.42 0)
+			(at 66.04 58.42 0)
 			(effects
 				(font
@@
 		)
 		(property "Description" "Power symbol creates a global label with name \"GND\" , ground"
-			(at 64.77 58.42 0)
+			(at 66.04 58.42 0)
 			(effects
 				(font
